File: projects/Monstera/Monstera.kicad_pcb (KiCad board)
At the start: 2 copper layers, 15.2 x 6.7 mm, 152 parts, among them J1 USB_C_Receptacle, SW1 SW_Push, U1 ATmega32U4-AU, Y1 16MHz

Commit message: Place everything
Parts:
- moved C5 28.8 mm to (309.6, 150.0), turned to 180 degrees
- moved C4 24.1 mm to (309.6, 146.8), turned to 180 degrees
- moved C3 20.0 mm to (309.6, 143.7), turned to 180 degrees
- moved SW1 17.4 mm to (307.2, 132.6)
- moved DS1 17.4 mm to (327.0, 136.5), turned to 90 degrees
- moved C2 16.8 mm to (309.6, 140.5), turned to 180 degrees
- moved C7 13.0 mm to (317.5, 154.8)
- moved R6 9.26 mm to (316.7, 135.7), turned to 90 degrees
- moved C6 8.87 mm to (323.9, 154.8)
- moved Y1 8.55 mm to (320.7, 154.8), turned to 90 degrees
- moved R5 8.09 mm to (323.9, 135.7), turned to 270 degrees
- moved J1 7.82 mm to (320.7, 124.6)
- moved C1 7.82 mm to (312.7, 145.3)
- moved R1 7.82 mm to (328.6, 145.3)
- moved U1 7.82 mm to (320.7, 145.3)
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
Commit message: Edge cuts!
Other:
- board size 15.2 x 6.7 mm -> 308 x 108.7 mm
